File: ad8342evb v1/ad8342evb v1.kicad_pcb (KiCad board)
At the start: 4 copper layers, 100 x 100 mm, 94 parts, among them J1 PWR_in_direct, J10 Bat, J11 3V3, J12 PWR_Jumper, J13 TP1, J14 TP1, J15 TP_PWR, J16 TP2, J17 TP3, J2 RF_in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

Commit message: added separate GNDA plane
Parts:
- added FB2: Ferrite_Bead, Inductor_SMD:L_0805_2012Metric_Pad1.15x1.40mm_HandSolder, F.Cu at (145.7, 109.8)
- added REF**: MountingHole_3.2mm_M3, MountingHole:MountingHole_3.2mm_M3, F.Cu at (195.0, 145.0)
- added REF**: MountingHole_3.2mm_M3, MountingHole:MountingHole_3.2mm_M3, F.Cu at (105.0, 145.0)
- added REF**: MountingHole_3.2mm_M3, MountingHole:MountingHole_3.2mm_M3, F.Cu at (105.0, 55.0)
- added REF**: MountingHole_3.2mm_M3, MountingHole:MountingHole_3.2mm_M3, F.Cu at (195.0, 55.0)
- moved D3 32.5 mm to (197.1, 115.6), turned to 270 degrees
- moved R32 28.2 mm to (197.1, 119.7), turned to 90 degrees
- moved J11 0.69 mm to (194.1, 138.1), turned to 180 degrees
Connections:
- C11 pad 2: GND -> GNDA
- C12 pad 1: GND -> GNDA
- C13 pad 2: GND -> GNDA
- C16 pad 2: GND -> GNDA
- C17 pad 1: GND -> GNDA
- C19 pad 2: GND -> GNDA
- C2 pad 2: GND -> GNDA
- C29 pad 2: GND -> GNDA
- C3 pad 2: GND -> GNDA
- C30 pad 2: GND -> GNDA
- C31 pad 2: GND -> GNDA
- C6 pad 2: GND -> GNDA
- C7 pad 2: GND -> GNDA
- C8 pad 2: GND -> GNDA
- C9 pad 2: GND -> GNDA
- D2 pad 1: GND -> GNDA
- J13 pad 2: GND -> GNDA
- J14 pad 1: GND -> GNDA
- J15 pad 1: GND -> GNDA
- J16 pad 1: GND -> GNDA
- J17 pad 1: GND -> GNDA
- J2 pad 2: GND -> GNDA
- J3 pad 2: GND -> GNDA
- J5 pad 2: GND -> GNDA
- R13 pad 2: GND -> GNDA
- R14 pad 2: GND -> GNDA
- R15 pad 2: GND -> GNDA
- R16 pad 2: GND -> GNDA
- R2 pad 1: GND -> GNDA
- R9 pad 1: GND -> GNDA
- U2 pad 4: GND -> GNDA
- U4 pad 11: GND -> GNDA
- U4 pad 13: GND -> GNDA
- U4 pad 17: GND -> GNDA
- U4 pad 4: GND -> GNDA
- U4 pad 5: GND -> GNDA
- U4 pad 8: GND -> GNDA
- U4 pad 9: GND -> GNDA
Routing:
- net GNDA: track 0.00 -> 47.9 mm, vias 0 -> 25
- net GND: track 80.1 -> 40.0 mm, vias 42 -> 23
- net Net-(F1-Pad2): track 67.0 -> 48.5 mm, vias 0 -> 2
- net /3V3: track 19.2 -> 23.3 mm, vias 2 -> 0
- added copper zone on In1.Cu, net GNDA

Commit message: fixed some bugs
Parts:
- removed REF** (x4): MountingHole_3.2mm_M3, MountingHole:MountingHole_3.2mm_M3
- R27: value 77K -> 75K
- moved C25 9.08 mm to (172.7, 119.4), turned to 180 degrees
- moved C21 4.90 mm to (181.5, 132.3), turned to 270 degrees
Connections:
- C23 pad 2: GND -> Net-(C23-Pad2)
- C25 pad 2: GND -> Net-(C23-Pad2)
- J10 pad 1: Net-(J10-Pad1) -> Net-(C21-Pad1)
- R28 pad 2: Net-(J10-Pad1) -> Net-(C21-Pad1)
- U3 pad 14: Net-(U3-Pad14) -> Net-(C23-Pad2)
- U3 pad 2: Net-(J10-Pad1) -> Net-(C21-Pad1)
Routing:
- net Net-(C21-Pad1): track 3.65 -> 38.6 mm, vias 1 -> 3
- net Net-(J10-Pad1): track 30.3 -> 0.00 mm, vias 2 -> 0
- net Net-(C23-Pad2): track 0.00 -> 13.9 mm, vias 0 -> 1
- net GND: track 40.0 -> 37.8 mm, vias 23 -> 21
- net Net-(R23-Pad1): track 14.8 -> 16.2 mm
Other:
- board text added: "AD8342 + LTC3558 Evaluation Board Version 1.1 Copyright 2020 Benjamin Menkuec"
- board text removed: "AD8342 + LTC3558 Evaluation Board Version 1.0 Copyright 2020 Benjamin Menkuec"
