File: ad8342evb v1/ad8342evb v1.sch (KiCad schematic (older format))
At the start: 95 parts, among them J1 PWR_in_direct, J10 Bat, J11 3V3, J12 PWR_Jumper, J13 TP1, J14 TP1, J15 TP_PWR, J16 TP2, J17 TP3, J2 RF_in, J3 LO_in, J4 Gain_Jumper, J5 IF_out, J6 PWR_in_switching, J7 PWR_in_USB, J8 PWR_in_LDO, J9 Mode_Jumper, U1 LM7805_TO220, U2 OPA2320, U3 LTC3558, U4 AD8342

Commit message: fixed some bugs
Parts:
- R27: value 77K -> 75K
Connections:
- net GND: no longer C23.2, C25.2
- net at U3.14 (V_C2): now also C23.2, C25.2
- net at J10.1 (Pin_1), R28.2, U3.2 (BAT): now also C21.1, U3.7 (PV_IN1), U3.8 (PV_IN2)
Changed lines of the file:
@@
 U 1 1 5F1D7C34
 P 8100 3000
-F 0 "U2" H 8100 3367 50  0000 C CNN
-F 1 "OPA2320" H 8100 3276 50  0000 C CNN
+F 0 "U2" H 8100 3300 50  0000 C CNN
+F 1 "OPA2320" H 8200 3200 50  0000 C CNN
 F 2 "Package_SO:SOIC-8_3.9x4.9mm_P1.27mm" H 8100 3000 50  0001 C CNN
 F 3 "http://www.ti.com/lit/ds/symlink/opa2320.pdf" H 8100 3000 50  0001 C CNN
@@
 	3650 5650 3900 5650
 Wire Wire Line
-	3900 5450 4150 5450
+	3900 5450 4000 5450
 Connection ~ 3650 5650
 $Comp
@@
 	4500 4750 4800 4750
 Wire Wire Line
-	3650 5300 4500 5300
+	3650 5300 4000 5300
 Connection ~ 4500 5300
 Wire Wire Line
@@
 F 3 "~" H 3850 7300 50  0001 C CNN
 	1    3850 7300
-	1    0    0    -1
-$EndComp
-$Comp
-L power:GND #PWR0139
-U 1 1 5F485E52
-P 3850 7650
-F 0 "#PWR0139" H 3850 7400 50  0001 C CNN
-F 1 "GND" H 3855 7477 50  0000 C CNN
-F 2 "" H 3850 7650 50  0001 C CNN
-F 3 "" H 3850 7650 50  0001 C CNN
-	1    3850 7650
 	1    0    0    -1
 $EndComp
@@
 $EndComp
 Wire Wire Line
-	4200 7650 3850 7650
-Wire Wire Line
 	6450 5450 6750 5450
 Wire Wire Line
@@
 P 4200 7200
 F 0 "R27" H 4270 7246 50  0000 L CNN
-F 1 "77K" H 4270 7155 50  0000 L CNN
+F 1 "75K" H 4270 7155 50  0000 L CNN
 F 2 "Resistor_SMD:R_0805_2012Metric_Pad1.15x1.40mm_HandSolder" V 4130 7200 50  0001 C CNN
 F 3 "~" H 4200 7200 50  0001 C CNN
@@
 Wire Wire Line
 	4700 7650 4200 7650
-Connection ~ 4200 7650
 $Comp
 L Device:R R23
@@
 Wire Wire Line
 	3850 7000 3850 7150
-Wire Wire Line
-	3850 7450 3850 7650
-Connection ~ 3850 7650
 Text Notes 4100 7750 0    50   ~ 0
 Filter values are estimates
@@
 $EndComp
 $Comp
-L power:GNDA #PWR?
+L power:GNDA #PWR0114
 U 1 1 5F699CE5
 P 7250 5900
-F 0 "#PWR?" H 7250 5650 50  0001 C CNN
+F 0 "#PWR0114" H 7250 5650 50  0001 C CNN
 F 1 "GNDA" H 7255 5727 50  0000 C CNN
 F 2 "" H 7250 5900 50  0001 C CNN
@@
 $EndComp
 $Comp
-L power:GNDA #PWR?
+L power:GNDA #PWR0152
 U 1 1 5F6C65F2
 P 8600 5850
-F 0 "#PWR?" H 8600 5600 50  0001 C CNN
+F 0 "#PWR0152" H 8600 5600 50  0001 C CNN
 F 1 "GNDA" H 8605 5677 50  0000 C CNN
 F 2 "" H 8600 5850 50  0001 C CNN
@@
 Wire Wire Line
 	7250 5900 7450 5900
+Wire Wire Line
+	4000 5450 4000 5300
+Connection ~ 4000 5450
+Wire Wire Line
+	4000 5450 4150 5450
+Connection ~ 4000 5300
+Wire Wire Line
+	4000 5300 4500 5300
+$Comp
+L power:GND #PWR0139
+U 1 1 5F485E52
+P 3850 7500
+F 0 "#PWR0139" H 3850 7250 50  0001 C CNN
+F 1 "GND" H 3855 7327 50  0000 C CNN
+F 2 "" H 3850 7500 50  0001 C CNN
+F 3 "" H 3850 7500 50  0001 C CNN
+	1    3850 7500
+	1    0    0    -1
+$EndComp
+Wire Wire Line
+	3850 7450 3850 7500
+Wire Wire Line
+	4200 7650 4000 7650
+Wire Wire Line
+	4000 7650 4000 7750
+Wire Wire Line
+	4000 7750 3650 7750
+Wire Wire Line
+	3650 7750 3650 6850
+Connection ~ 4200 7650
 $EndSCHEMATC
