File: ad8342evb.kicad_pcb (KiCad board)
At the start: 4 copper layers, 100 x 100 mm, 97 parts, among them J1 PWR_in_direct, J10 Bat, J11 3V3, J12 PWR_Jumper, J13 TP1, J14 TP1, J15 TP_PWR, J16 TP2, J17 TP3, J2 RF_in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

Commit message: added more decoupling caps
Parts:
- added C32: 1uF, Capacitor_SMD:C_0805_2012Metric_Pad1.15x1.40mm_HandSolder, F.Cu at (144.8, 64.7)
- added C33: 1uF, Capacitor_SMD:C_0805_2012Metric_Pad1.15x1.40mm_HandSolder, F.Cu at (146.7, 82.7)
- C10, C14, C15, C18, C3, C4, C9: value 10uF -> 1uF
- R34: value 10k -> 100
Routing:
- net GNDA: track 47.1 -> 52.3 mm, vias 25 -> 29
- net +5V: track 29.4 -> 33.6 mm
Other:
- board text added: "Gain: low mid high"
- board text removed: "Gain: high mid low"
